File: Circuits/Sender/BicycleFinder.kicad_pcb (KiCad board)
At the start: 2 copper layers, 64.1 x 40.1 mm, 11 parts, among them CN1 WRITER, SW1 SW_PUSH, U1 LITE_LITE, U2 HN2S01FU

Commit message: Reviewed parts layout.
Parts:
- JP1, R1, R2, U2: moved to F.Cu
- U1: footprint TWE-001L-SMD-noNTH -> TWE-001L-SMD
- moved CN1 27.7 mm to (214.6, 148.8), turned to 0 degrees
- moved R1 26.3 mm to (188.5, 125.0), turned to 0 degrees
- moved R2 19.9 mm to (211.3, 128.0), turned to 90 degrees
- moved JP1 8.01 mm to (211.3, 125.2), turned to 180 degrees
- moved U2 4.71 mm to (213.9, 125.2), turned to 90 degrees
- turned LD1 to 270 degrees
- turned U1 to 270 degrees
Routing:
- net GND: track 0.00 -> 67.2 mm, vias 0 -> 1
- net /PRG: track 0.00 -> 43.7 mm
- net /Vcc: track 0.00 -> 42.1 mm, vias 0 -> 1
- net /M1: track 0.00 -> 38.7 mm, vias 0 -> 1
- net /RX: track 0.00 -> 32.7 mm
- net /TX: track 0.00 -> 31.9 mm
- net /LED: track 0.00 -> 29.9 mm
- net /DC3V: track 0.00 -> 28.7 mm, vias 0 -> 2
- net /CHG: track 0.00 -> 28.3 mm
- net /RST: track 0.00 -> 27.9 mm
- net /DO4: track 0.00 -> 20.1 mm
- net /DI1: track 0.00 -> 18.9 mm
- net /3V: track 0.00 -> 9.73 mm

Commit message: Moved some chip parts.
Parts:
- R1: value 560 -> 330
- R2: value 560 -> 680
- moved R2 186.3 mm to (43.7, 46.7), turned to 0 degrees
- moved BT1 183.7 mm to (27.9, 33.9)
- moved C1 183.7 mm to (77.5, 33.9)
- moved SW1 183.7 mm to (50.2, 33.9)
- moved U1 183.7 mm to (34.3, 33.9)
- moved CN1 183.7 mm to (62.2, 46.2)
- moved LD1 183.7 mm to (39.9, 45.1), turned to 180 degrees
- moved PBPS-85 183.7 mm to (48.5, 33.9)
- moved R1 183.7 mm to (36.1, 22.4)
- moved U2 181.3 mm to (62.5, 25.4), turned to 180 degrees
- moved JP1 180.9 mm to (62.5, 22.4), turned to 270 degrees
Routing:
- net /Vcc: track 42.1 -> 73.5 mm
- net /LED: track 29.9 -> 2.80 mm
- net /DC3V: track 28.7 -> 23.1 mm, vias 2 -> 0
- net /PRG: track 43.7 -> 47.8 mm
- net /DO4: track 20.1 -> 16.5 mm, vias 0 -> 1
- net /M1: track 38.7 -> 36.0 mm, vias 1 -> 0
- net /RX: track 32.7 -> 34.4 mm, vias 0 -> 1
- net /CHG: track 28.3 -> 29.7 mm
- net /RST: track 27.9 -> 27.0 mm
Other:
- outline, holes or cut-outs redrawn
- board text added: "CFG"
- board text added: "GND"
- board text added: "PRG"
- board text added: "RST"
- board text added: "RXD"
- board text added: "TXD"
- board text added: "Vcc"

Commit message: Moved pin names of writer to F.Silk layer.
Routing:
- net (no net): track 0.00 -> 5.21 mm, vias 0 -> 2
- added copper zone on F.Cu, net (none)
Changed lines of the file:
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@@
     (area 13.526699 13.529999 78.332401 54.288001)
     (thickness 1)
-    (drawings 7)
-    (tracks 103)
+    (drawings 9)
+    (tracks 106)
     (zones 0)
     (modules 11)
@@
     (pad_drill 2)
     (pad_to_mask_clearance 0)
-    (aux_axis_origin 162.56 113.03)
+    (aux_axis_origin 12.7 12.7)
     (visible_elements 7FFFFFFF)
     (pcbplotparams
-      (layerselection 287342593)
+      (layerselection 284196865)
       (usegerberextensions true)
       (excludeedgelayer true)
       (linewidth 0.150000)
       (plotframeref false)
-      (viasonmask true)
+      (viasonmask false)
       (mode 1)
-      (useauxorigin true)
+      (useauxorigin false)
       (hpglpennumber 1)
       (hpglpenspeed 20)
@@
       (psa4output false)
       (plotreference true)
-      (plotvalue false)
+      (plotvalue true)
       (plotothertext true)
       (plotinvisibletext false)
@@
     )
   )
-  (gr_text CFG (at 69.596 50.292 270) (layer F.Cu)
+  (dimension 64.516245 (width 0.3) (layer Eco2.User)
+    (gr_text 64.516mm (at 46.034859 62.123522 359.8420986) (layer Eco2.User)
+      (effects (font (size 1.5 1.5) (thickness 0.3)))
+    )
+    (feature1 (pts (xy 78.3717 33.6042) (xy 78.289139 63.562417)))
+    (feature2 (pts (xy 13.8557 33.4264) (xy 13.773139 63.384617)))
+    (crossbar (pts (xy 13.780579 60.684628) (xy 78.296579 60.862428)))
+    (arrow1a (pts (xy 78.296579 60.862428) (xy 77.168464 61.445741)))
+    (arrow1b (pts (xy 78.296579 60.862428) (xy 77.171696 60.272905)))
+    (arrow2a (pts (xy 13.780579 60.684628) (xy 14.905462 61.274151)))
+    (arrow2b (pts (xy 13.780579 60.684628) (xy 14.908694 60.101315)))
+  )
+  (dimension 40.132032 (width 0.3) (layer Eco2.User)
+    (gr_text 40.132mm (at 88.192733 33.886954 270.0725263) (layer Eco2.User)
+      (effects (font (size 1.5 1.5) (thickness 0.3)))
+    )
+    (feature1 (pts (xy 70.8025 53.975) (xy 89.568132 53.951246)))
+    (feature2 (pts (xy 70.7517 13.843) (xy 89.517332 13.819246)))
+    (crossbar (pts (xy 86.817335 13.822663) (xy 86.868135 53.954663)))
+    (arrow1a (pts (xy 86.868135 53.954663) (xy 86.280289 52.828903)))
+    (arrow1b (pts (xy 86.868135 53.954663) (xy 87.453129 52.827418)))
+    (arrow2a (pts (xy 86.817335 13.822663) (xy 86.232341 14.949908)))
+    (arrow2b (pts (xy 86.817335 13.822663) (xy 87.405181 14.948423)))
+  )
+  (gr_text CFG (at 69.596 50.292 270) (layer F.SilkS)
     (effects (font (size 1.5 1.5) (thickness 0.3)))
   )
-  (gr_text GND (at 67.056 50.292 270) (layer F.Cu)
+  (gr_text GND (at 67.056 50.292 270) (layer F.SilkS)
     (effects (font (size 1.5 1.5) (thickness 0.3)))
   )
-  (gr_text TXD (at 64.516 50.292 270) (layer F.Cu)
+  (gr_text TXD (at 64.516 50.292 270) (layer F.SilkS)
     (effects (font (size 1.5 1.5) (thickness 0.3)))
   )
-  (gr_text PRG (at 61.976 50.292 270) (layer F.Cu)
+  (gr_text PRG (at 61.976 50.292 270) (layer F.SilkS)
     (effects (font (size 1.5 1.5) (thickness 0.3)))
   )
-  (gr_text RXD (at 59.436 50.292 270) (layer F.Cu)
+  (gr_text RXD (at 59.436 50.292 270) (layer F.SilkS)
     (effects (font (size 1.5 1.5) (thickness 0.3)))
   )
-  (gr_text RST (at 56.896 50.292 270) (layer F.Cu)
+  (gr_text RST (at 56.896 50.292 270) (layer F.SilkS)
     (effects (font (size 1.5 1.5) (thickness 0.3)))
   )
-  (gr_text Vcc (at 54.356 50.292 270) (layer F.Cu)
+  (gr_text Vcc (at 54.356 50.292 270) (layer F.SilkS)
     (effects (font (size 1.5 1.5) (thickness 0.3)))
   )
+  (via (at 26.924 45.593) (size 0.889) (layers F.Cu B.Cu) (net 0))
+  (via (at 32.131 45.593) (size 0.889) (layers F.Cu B.Cu) (net 0))
+  (segment (start 26.924 45.593) (end 32.131 45.593) (width 0.254) (layer B.Cu) (net 0))
   (segment (start 29.2747 22.352) (end 27.94 21.0173) (width 0.508) (layer F.Cu) (net 1))
   (segment (start 35.306 22.352) (end 29.2747 22.352) (width 0.508) (layer F.Cu) (net 1))
@@
     (connect_pads (clearance 0.508))
     (min_thickness 0.254)
-    (keepout (tracks not_allowed) (vias not_allowed) (copperpour allowed))
-    (fill (arc_segments 16) (thermal_gap 0.508) (thermal_bridge_width 0.508))
-    (polygon
-      (pts
-        (xy 46.228 13.716) (xy 46.228 19.304) (xy 50.8 19.304) (xy 50.8 13.716)
-      )
-    )
+    (keepout (tracks not_allowed) (vias not_allowed) (copperpour not_allowed))
+    (fill (arc_segments 16) (thermal_gap 0.508) (thermal_bridge_width 0.508))
+    (polygon
+      (pts
+        (xy 46.355 13.97) (xy 46.355 19.558) (xy 50.673 19.558) (xy 50.673 13.97)
+      )
+    )
+  )
+  (zone (net 0) (net_name "") (layer F.Cu) (hatch edge 0.508)
+    (connect_pads (clearance 0.508))
+    (min_thickness 0.254)
+    (fill (arc_segments 16) (thermal_gap 0.508) (thermal_bridge_width 0.508))
+    (polygon
+      (pts
+        (xy 49.53 18.796) (xy 19.304 18.796) (xy 19.304 49.022) (xy 49.53 49.022)
+      )
+    )
+  )
+  (zone (net 0) (net_name "") (layer F.Cu) (hatch edge 0.508)
+    (connect_pads (clearance 0.508))
+    (min_thickness 0.254)
+    (keepout (tracks not_allowed) (vias not_allowed) (copperpour not_allowed))
+    (fill (arc_segments 16) (thermal_gap 0.508) (thermal_bridge_width 0.508))
+    (polygon
+      (pts
+        (xy 46.355 53.848) (xy 46.355 48.26) (xy 50.673 48.26) (xy 50.673 53.848)
+      )
+    )
+  )
+  (zone (net 0) (net_name "") (layer F.Cu) (hatch edge 0.508)
+    (connect_pads (clearance 0.508))
+    (min_thickness 0.254)
+    (keepout (tracks not_allowed) (vias not_allowed) (copperpour not_allowed))
+    (fill (arc_segments 16) (thermal_gap 0.508) (thermal_bridge_width 0.508))
+    (polygon
+      (pts
+        (xy 20.955 53.721) (xy 20.955 48.26) (xy 25.4 48.26) (xy 25.4 53.721)
+      )
+    )
+  )
+  (zone (net 0) (net_name "") (layer F.Cu) (hatch edge 0.508)
+    (connect_pads (clearance 0.508))
+    (min_thickness 0.254)
+    (keepout (tracks not_allowed) (vias not_allowed) (copperpour not_allowed))
+    (fill (arc_segments 16) (thermal_gap 0.508) (thermal_bridge_width 0.508))
+    (polygon
+      (pts
+        (xy 20.828 14.224) (xy 20.828 19.558) (xy 25.4 19.558) (xy 25.4 14.224)
+      )
+    )
+  )
+  (zone (net 0) (net_name "") (layer F.Cu) (hatch edge 0.508)
+    (connect_pads (clearance 0.508))
+    (min_thickness 0.254)
+    (keepout (tracks not_allowed) (vias not_allowed) (copperpour not_allowed))
+    (fill (arc_segments 16) (thermal_gap 0.508) (thermal_bridge_width 0.508))
+    (polygon
+      (pts
+        (xy 27.559 28.067) (xy 30.988 28.067) (xy 30.988 32.639) (xy 27.559 32.639)
+      )
+    )
